File: famicom-to-nes.kicad_pcb (KiCad board)
At the start: 2 copper layers, 99.7 x 40.9 mm, 5 parts, among them J1 NES, J2 Famicom, U1 AVR CIC

Commit message: Rev 1.2
Parts:
- moved REF** 45.4 mm to (187.0, 84.1)
- moved C1 0.13 mm to (98.7, 82.7)
- moved U1 0.13 mm to (93.3, 86.0)
- moved J1 0.13 mm to (141.5, 106.8)
- moved J2 0.13 mm to (182.7, 65.6)
Routing:
- net /RW: track 21.7 -> 29.8 mm, vias 1 -> 3
- net /A3: track 21.8 -> 29.7 mm, vias 1 -> 3
- net /D5: track 22.1 -> 29.9 mm, vias 1 -> 3
- net /PHI2: track 22.2 -> 29.7 mm, vias 1 -> 3
- net /A6: track 21.2 -> 28.6 mm, vias 1 -> 3
- net +5V: track 110.1 -> 117.4 mm, vias 0 -> 1
- net /D6: track 22.6 -> 29.9 mm, vias 1 -> 3
- net /A7: track 21.6 -> 28.7 mm, vias 1 -> 3
- net /PRG: track 23.3 -> 30.2 mm, vias 1 -> 3
- net /D3: track 23.3 -> 30.0 mm, vias 1 -> 3
- net /D7: track 23.2 -> 29.8 mm, vias 1 -> 3
- net /4MHz: track 18.7 -> 25.2 mm, vias 0 -> 2
- net /D0: track 23.7 -> 30.1 mm, vias 1 -> 3
- net /A4: track 23.2 -> 29.6 mm, vias 1 -> 3
- net /D1: track 23.8 -> 30.1 mm, vias 1 -> 3
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Other:
- board text added: "Famicom to NES Converter Rev 1.2 (Nov) Yaroslav Veremenko (c) 2022 https://github.com/veremenko-y/famicom-to-nes"
- board text added: "PIN 1"
- board text added: "To change region, press reset 4-8 times."
- board text removed: "Famicom to NES Converter Rev 1.1 (Nov) Yaroslav Veremenko (c) 2022 https://github.com/veremenko-y/famicom-to-nes"
